File: hw/ML0/ML0.kicad_sch (KiCad schematic)
At the start: 0 parts

Commit message: Working on V0 of the analog PCB
Parts:
- added H1, H2, H3, H4: MountingHole, symbol Mechanical:MountingHole
- added J1: Rig Connector, symbol Connector_Generic:Conn_01x06
- added J2: 12V Supply, symbol Connector_Generic:Conn_01x02
- added J3: Digital Connector, symbol Connector_Generic:Conn_01x05
- added J4: ADC Connector, symbol Connector_Generic:Conn_01x02
Connections:
- new net +12V: J2.1 (Pin_1)
- new net ADC0: J4.1 (Pin_1)
- new net GNDA: J2.2 (Pin_2), J3.5 (Pin_5), J4.2 (Pin_2)
- new net GPIO_COS: J3.3 (Pin_3)
- new net GPIO_PTT: J3.4 (Pin_4)
- new net IC20_SCL: J3.2 (Pin_2)
- new net IC20_SDA: J3.1 (Pin_1)
- new net RIG_AF_IN: J1.2 (Pin_2)
- new net RIG_AF_OUT: J1.4 (Pin_4)
- new net RIG_GND: J1.1 (Pin_1), J1.3 (Pin_3), J1.5 (Pin_5)
- new net RIG_PTT: J1.6 (Pin_6)

Commit message: Working on PCB 0
Parts:
- H1, H2, H3, H4: footprint (none) -> MountingHole:MountingHole_4mm
- J1: footprint (none) -> Connector_PinHeader_2.54mm:PinHeader_1x06_P2.54mm_Vertical
- J2: footprint (none) -> Connector_PinHeader_2.54mm:PinHeader_1x02_P2.54mm_Vertical
- J3: footprint (none) -> Connector_PinHeader_2.54mm:PinHeader_1x05_P2.54mm_Vertical
- J4: footprint (none) -> Connector_Wire:SolderWire-2.5sqmm_1x02_P7.2mm_D2.4mm_OD3.6mm_Relief
Changed lines of the file:
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@@
       (effects (font (size 1.27 1.27)))
     )
-    (property "Footprint" "" (at 205.74 67.31 0)
+    (property "Footprint" "Connector_PinHeader_2.54mm:PinHeader_1x06_P2.54mm_Vertical" (at 205.74 67.31 0)
       (effects (font (size 1.27 1.27)) hide)
     )
@@
       (effects (font (size 1.27 1.27)) (justify left))
     )
-    (property "Footprint" "" (at 240.03 90.17 0)
+    (property "Footprint" "Connector_PinHeader_2.54mm:PinHeader_1x05_P2.54mm_Vertical" (at 240.03 90.17 0)
       (effects (font (size 1.27 1.27)) hide)
     )
@@
       (effects (font (size 1.27 1.27)) (justify left))
     )
-    (property "Footprint" "" (at 139.7 93.98 0)
+    (property "Footprint" "MountingHole:MountingHole_4mm" (at 139.7 93.98 0)
       (effects (font (size 1.27 1.27)) hide)
     )
@@
       (effects (font (size 1.27 1.27)))
     )
-    (property "Footprint" "" (at 212.09 137.16 0)
+    (property "Footprint" "Connector_PinHeader_2.54mm:PinHeader_1x02_P2.54mm_Vertical" (at 212.09 137.16 0)
       (effects (font (size 1.27 1.27)) hide)
     )
@@
       (effects (font (size 1.27 1.27)) (justify left))
     )
-    (property "Footprint" "" (at 139.7 109.22 0)
+    (property "Footprint" "MountingHole:MountingHole_4mm" (at 139.7 109.22 0)
       (effects (font (size 1.27 1.27)) hide)
     )
@@
       (effects (font (size 1.27 1.27)) (justify left))
     )
-    (property "Footprint" "" (at 240.03 111.76 0)
+    (property "Footprint" "Connector_Wire:SolderWire-2.5sqmm_1x02_P7.2mm_D2.4mm_OD3.6mm_Relief" (at 240.03 111.76 0)
       (effects (font (size 1.27 1.27)) hide)
     )
@@
       (effects (font (size 1.27 1.27)) (justify left))
     )
-    (property "Footprint" "" (at 139.7 101.6 0)
+    (property "Footprint" "MountingHole:MountingHole_4mm" (at 139.7 101.6 0)
       (effects (font (size 1.27 1.27)) hide)
     )
@@
       (effects (font (size 1.27 1.27)) (justify left))
     )
-    (property "Footprint" "" (at 139.7 116.84 0)
-      (effects (font (size 1.27 1.27)) hide)
-    )
+    (property "Footprint" "MountingHole:MountingHole_4mm" (at 139.7 116.84 0)
+      (effects (font (size 1.27 1.27)) hide)
+    )

Commit message: Docs
Parts:
- removed J1: Rig Connector, Connector_PinHeader_2.54mm:PinHeader_1x06_P2.54mm_Vertical, symbol Connector_Generic:Conn_01x06
- added J1: Rig Connector, Connector_PinHeader_2.54mm:PinHeader_1x07_P2.54mm_Vertical, symbol Connector_Generic:Conn_01x07
- J4: footprint Connector_Wire:SolderWire-2.5sqmm_1x02_P7.2mm_D2.4mm_OD3.6mm_Relief -> Connector_PinHeader_2.54mm:PinHeader_1x02_P2.54mm_Vertical
Connections:
- net RIG_AF_IN: now also J1.2 (Pin_2)
- net RIG_AF_OUT: now also J1.4 (Pin_4)
- net RIG_GND: now also J1.1 (Pin_1), J1.3 (Pin_3), J1.5 (Pin_5)
- net RIG_PTT: now also J1.6 (Pin_6)
- new net RIG_COS: J1.7 (Pin_7)
Changed lines of the file:
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@@
+    (stroke (width 0) (type default))
+  )
+  (wire (pts (xy 210.82 77.47) (xy 226.06 77.47))
     (stroke (width 0) (type default))
   )
@@
     )
   )
+  (global_label "RIG_COS" (shape input) (at 226.06 77.47 0) (fields_autoplaced)
+    (effects (font (size 1.27 1.27)) (justify left))
+    (property "Intersheetrefs" "${INTERSHEET_REFS}" (at 236.9676 77.47 0)
+      (effects (font (size 1.27 1.27)) (justify left) hide)
+    )
+  )
   (global_label "RIG_GND" (shape input) (at 226.06 62.23 0) (fields_autoplaced)
     (effects (font (size 1.27 1.27)) (justify left))
@@
         (path "/5f8f636b-fd0e-498e-8696-0a023acb4c09"
           (reference "#PWR023") (unit 1)
-        )
-      )
-    )
-  )
-  (symbol (lib_id "Connector_Generic:Conn_01x06") (at 205.74 67.31 0) (mirror y) (unit 1)
-    (in_bom yes) (on_board yes) (dnp no) (fields_autoplaced)
-    (property "Reference" "J1" (at 205.74 55.88 0)
-      (effects (font (size 1.27 1.27)))
-    )
-    (property "Value" "Rig Connector" (at 205.74 58.42 0)
-      (effects (font (size 1.27 1.27)))
-    )
-    (property "Footprint" "Connector_PinHeader_2.54mm:PinHeader_1x06_P2.54mm_Vertical" (at 205.74 67.31 0)
-      (effects (font (size 1.27 1.27)) hide)
-    )
-    (property "Datasheet" "~" (at 205.74 67.31 0)
-      (effects (font (size 1.27 1.27)) hide)
-    )
-    (pin "1")
-    (pin "4")
-    (pin "3")
-    (pin "2")
-    (pin "6")
-    (pin "5")
-    (instances
-      (project "ML0"
-        (path "/5f8f636b-fd0e-498e-8696-0a023acb4c09"
-          (reference "J1") (unit 1)
         )
       )
@@
     )
   )
+  (symbol (lib_id "Connector_Generic:Conn_01x07") (at 205.74 69.85 0) (mirror y) (unit 1)
+    (in_bom yes) (on_board yes) (dnp no) (fields_autoplaced)
+    (property "Reference" "J1" (at 205.74 55.88 0)
+      (effects (font (size 1.27 1.27)))
+    )
+    (property "Value" "Rig Connector" (at 205.74 58.42 0)
+      (effects (font (size 1.27 1.27)))
+    )
+    (property "Footprint" "Connector_PinHeader_2.54mm:PinHeader_1x07_P2.54mm_Vertical" (at 205.74 69.85 0)
+      (effects (font (size 1.27 1.27)) hide)
+    )
+    (property "Datasheet" "~" (at 205.74 69.85 0)
+      (effects (font (size 1.27 1.27)) hide)
+    )
+    (pin "5")
+    (pin "7")
+    (pin "6")
+    (pin "3")
+    (pin "2")
+    (pin "1")
+    (pin "4")
+    (instances
+      (project "ML0"
+        (path "/5f8f636b-fd0e-498e-8696-0a023acb4c09"
+          (reference "J1") (unit 1)
+        )
+      )
+    )
+  )
   (symbol (lib_id "Mechanical:MountingHole") (at 139.7 93.98 0) (unit 1)
     (in_bom yes) (on_board yes) (dnp no) (fields_autoplaced)
@@
       (effects (font (size 1.27 1.27)) (justify left))
     )
-    (property "Footprint" "Connector_Wire:SolderWire-2.5sqmm_1x02_P7.2mm_D2.4mm_OD3.6mm_Relief" (at 240.03 111.76 0)
-      (effects (font (size 1.27 1.27)) hide)
-    )
+    (property "Footprint" "Connector_PinHeader_2.54mm:PinHeader_1x02_P2.54mm_Vertical" (at 240.03 111.76 0)
+      (effects (font (size 1.27 1.27)) hide)
+    )

Commit message: Initial layout done
Parts:
- removed J1: Rig Connector, Connector_PinHeader_2.54mm:PinHeader_1x07_P2.54mm_Vertical, symbol Connector_Generic:Conn_01x07
- added J1: Conn_01x06, Connector_PinHeader_2.54mm:PinHeader_1x06_P2.54mm_Vertical, symbol Connector_Generic:Conn_01x06
Connections:
- net GPIO_COS: now also J3.1 (Pin_1); no longer J3.3 (Pin_3)
- net GPIO_PTT: now also J3.2 (Pin_2); no longer J3.4 (Pin_4)
- net IC20_SCL: now also J3.4 (Pin_4); no longer J3.2 (Pin_2)
- net IC20_SDA: now also J3.3 (Pin_3); no longer J3.1 (Pin_1)
- net RIG_AF_IN: now also J1.6 (Pin_6)
- net RIG_COS: now also J1.3 (Pin_3)
- net RIG_GND: now also J1.4 (Pin_4)
- net RIG_PTT: now also J1.5 (Pin_5)
- new net RIG_AF_OUT+: J1.1 (Pin_1)
- new net RIG_AF_OUT-: J1.2 (Pin_2)
