File: hw/ML0/Power.kicad_sch (KiCad schematic)
At the start: 0 parts

Commit message: Working on V0 of the analog PCB
Parts:
- added C7, C8: 10u, symbol Device:C_Polarized_Small_US
- added D1: LED, symbol Device:LED
- added R7: R_Small_US, symbol Device:R_Small_US
- added U3: NCP1117-3.3_SOT223, Package_TO_SOT_SMD:SOT-223-3_TabPin2, symbol Regulator_Linear:NCP1117-3.3_SOT223
Connections:
- new net: D1.2 (A), R7.2
- new net +12V: C8.1, U3.3 (VI)
- new net +3.3VA: C7.1, R7.1, U3.2 (VO)
- new net GNDA: C7.2, C8.2, D1.1 (K), U3.1 (GND)
Other:
- company: (none) -> Bruce MacKinnon KC1FSZ
- title: (none) -> MicroLink - Power Related

Commit message: Working on PCB 0
Parts:
- C7, C8: footprint (none) -> Capacitor_SMD:CP_Elec_8x10
- D1: footprint (none) -> LED_SMD:LED_0805_2012Metric_Pad1.15x1.40mm_HandSolder
- R7: value R_Small_US -> 220; footprint (none) -> Resistor_SMD:R_0805_2012Metric_Pad1.20x1.40mm_HandSolder
Changed lines of the file:
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@@
       (effects (font (size 1.27 1.27)) (justify left))
     )
-    (property "Footprint" "" (at 80.01 86.36 0)
+    (property "Footprint" "Capacitor_SMD:CP_Elec_8x10" (at 80.01 86.36 0)
       (effects (font (size 1.27 1.27)) hide)
     )
@@
       (effects (font (size 1.27 1.27)) (justify left))
     )
-    (property "Footprint" "" (at 123.19 85.09 0)
+    (property "Footprint" "Capacitor_SMD:CP_Elec_8x10" (at 123.19 85.09 0)
       (effects (font (size 1.27 1.27)) hide)
     )
@@
       (effects (font (size 1.27 1.27)) (justify left))
     )
-    (property "Value" "R_Small_US" (at 142.24 78.74 0)
+    (property "Value" "220" (at 142.24 78.74 0)
       (effects (font (size 1.27 1.27)) (justify left))
     )
-    (property "Footprint" "" (at 139.7 77.47 0)
+    (property "Footprint" "Resistor_SMD:R_0805_2012Metric_Pad1.20x1.40mm_HandSolder" (at 139.7 77.47 0)
       (effects (font (size 1.27 1.27)) hide)
     )
@@
       (effects (font (size 1.27 1.27)) (justify right))
     )
-    (property "Footprint" "" (at 139.7 83.82 0)
+    (property "Footprint" "LED_SMD:LED_0805_2012Metric_Pad1.15x1.40mm_HandSolder" (at 139.7 83.82 0)
       (effects (font (size 1.27 1.27)) hide)
     )

Commit message: Docs
Parts:
- C7, C8: footprint Capacitor_SMD:CP_Elec_8x10 -> Capacitor_SMD:CP_Elec_5x5.3
Changed lines of the file:
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@@
       (effects (font (size 1.27 1.27)) (justify left))
     )
-    (property "Footprint" "Capacitor_SMD:CP_Elec_8x10" (at 80.01 86.36 0)
+    (property "Footprint" "Capacitor_SMD:CP_Elec_5x5.3" (at 80.01 86.36 0)
       (effects (font (size 1.27 1.27)) hide)
     )
@@
       (effects (font (size 1.27 1.27)) (justify left))
     )
-    (property "Footprint" "Capacitor_SMD:CP_Elec_8x10" (at 123.19 85.09 0)
+    (property "Footprint" "Capacitor_SMD:CP_Elec_5x5.3" (at 123.19 85.09 0)
       (effects (font (size 1.27 1.27)) hide)
     )

Commit message: Initial layout done
Parts:
- C7, C8: footprint Capacitor_SMD:CP_Elec_5x5.3 -> KiCad-Library:CAP_KEMET_530_530
Changed lines of the file:
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@@
       (effects (font (size 1.27 1.27)) (justify left))
     )
-    (property "Footprint" "Capacitor_SMD:CP_Elec_5x5.3" (at 80.01 86.36 0)
+    (property "Footprint" "KiCad-Library:CAP_KEMET_530_530" (at 80.01 86.36 0)
       (effects (font (size 1.27 1.27)) hide)
     )
@@
       (effects (font (size 1.27 1.27)) (justify left))
     )
-    (property "Footprint" "Capacitor_SMD:CP_Elec_5x5.3" (at 123.19 85.09 0)
+    (property "Footprint" "KiCad-Library:CAP_KEMET_530_530" (at 123.19 85.09 0)
       (effects (font (size 1.27 1.27)) hide)
     )
