File: hw/ML0/AudioOut.kicad_sch (KiCad schematic)
At the start: 13 parts, among them T1 Transformer_1P_1S, U1 LMV321, U2 LTV-356T

Commit message: Working on V0 of the analog PCB
Parts:
- added C5: 0.1u, symbol Device:C_Small
- added C6: 4.7u, symbol Device:C_Polarized_Small_US
- added C9: 10u, symbol Device:C_Polarized_Small_US
- added JP1: DAC Address Control, symbol Jumper:SolderJumper_2_Bridged
- added JP2: SolderJumper_2_Open, symbol Jumper:SolderJumper_2_Open
- added R5, R6: 10k, symbol Device:R_Small_US
- added U4: MCP4725xxx-xCH, Package_TO_SOT_SMD:SOT-23-6, symbol Analog_DAC:MCP4725xxx-xCH
Connections:
- net GND is gone; now on net GNDA: U2.2
- net +3.3VA: now also C5.1, C9.1, JP2.2 (B), R5.1, R6.1, U4.3 (VDD)
- net GNDA: now also C5.2, C9.2, JP1.1 (A), U4.2 (VSS)
- net at C3.2, TP1.1, U1.3 (-)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: now also C6.1; no longer R3.1
- net DAC0: no longer names the net of R1.2
- net DAC0: now also U4.1 (VOUT)
- new net: C6.2, R3.1
- new net: JP1.2 (B), JP2.1 (A), U4.6 (A0)
- new net IC20_SCL: R6.2, U4.5 (SCL)
- new net IC20_SDA: R5.2, U4.4 (SDA)
Other:
- note added: "DAC"
- moved on the sheet: C1, C2, C3, C4, R1, R2, R3, R4, RV1, T1, TP1, U1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

Commit message: Working on PCB 0
Parts:
- C1, C6, C9: footprint (none) -> Capacitor_SMD:CP_Elec_8x10
- C2, C3, C4, C5: footprint (none) -> Capacitor_SMD:C_0805_2012Metric_Pad1.18x1.45mm_HandSolder
- JP1: footprint (none) -> Jumper:SolderJumper-2_P1.3mm_Bridged_Pad1.0x1.5mm
- JP2: footprint (none) -> Jumper:SolderJumper-2_P1.3mm_Open_Pad1.0x1.5mm
- R1: value 2.2k -> 1.5k; footprint (none) -> Resistor_SMD:R_0805_2012Metric_Pad1.20x1.40mm_HandSolder
- R2: value 3.9k -> 2.7k; footprint (none) -> Resistor_SMD:R_0805_2012Metric_Pad1.20x1.40mm_HandSolder
- R3, R4, R5, R6: footprint (none) -> Resistor_SMD:R_0805_2012Metric_Pad1.20x1.40mm_HandSolder
Changed lines of the file:
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@@
       (effects (font (size 1.27 1.27)))
     )
-    (property "Footprint" "" (at 177.8 86.36 0)
+    (property "Footprint" "Capacitor_SMD:CP_Elec_8x10" (at 177.8 86.36 0)
       (effects (font (size 1.27 1.27)) hide)
     )
@@
       (effects (font (size 1.27 1.27)) (justify left))
     )
-    (property "Footprint" "" (at 46.99 55.88 0)
+    (property "Footprint" "Resistor_SMD:R_0805_2012Metric_Pad1.20x1.40mm_HandSolder" (at 46.99 55.88 0)
       (effects (font (size 1.27 1.27)) hide)
     )
@@
       (effects (font (size 1.27 1.27)) (justify left))
     )
-    (property "Footprint" "" (at 99.06 59.69 0)
+    (property "Footprint" "Capacitor_SMD:C_0805_2012Metric_Pad1.18x1.45mm_HandSolder" (at 99.06 59.69 0)
       (effects (font (size 1.27 1.27)) hide)
     )
@@
       (effects (font (size 1.27 1.27)) (justify left))
     )
-    (property "Footprint" "" (at 57.15 60.96 0)
+    (property "Footprint" "Resistor_SMD:R_0805_2012Metric_Pad1.20x1.40mm_HandSolder" (at 57.15 60.96 0)
       (effects (font (size 1.27 1.27)) hide)
     )
@@
       (effects (font (size 1.27 1.27)) (justify right) hide)
     )
-    (property "Footprint" "" (at 60.96 74.93 0)
+    (property "Footprint" "Jumper:SolderJumper-2_P1.3mm_Open_Pad1.0x1.5mm" (at 60.96 74.93 0)
       (effects (font (size 1.27 1.27)) hide)
     )
@@
       (effects (font (size 1.27 1.27)) (justify left))
     )
-    (property "Footprint" "" (at 140.6652 106.68 0)
+    (property "Footprint" "Capacitor_SMD:C_0805_2012Metric_Pad1.18x1.45mm_HandSolder" (at 140.6652 106.68 0)
       (effects (font (size 1.27 1.27)) hide)
     )
@@
       (effects (font (size 1.27 1.27)))
     )
-    (property "Footprint" "" (at 207.264 137.414 90)
+    (property "Footprint" "Resistor_SMD:R_0805_2012Metric_Pad1.20x1.40mm_HandSolder" (at 207.264 137.414 90)
       (effects (font (size 1.27 1.27)) hide)
     )
@@
       (effects (font (size 1.27 1.27)))
     )
-    (property "Value" "2.2k" (at 111.76 80.01 90)
-      (effects (font (size 1.27 1.27)))
-    )
-    (property "Footprint" "" (at 111.506 84.836 90)
+    (property "Value" "1.5k" (at 111.76 80.01 90)
+      (effects (font (size 1.27 1.27)))
+    )
+    (property "Footprint" "Resistor_SMD:R_0805_2012Metric_Pad1.20x1.40mm_HandSolder" (at 111.506 84.836 90)
       (effects (font (size 1.27 1.27)) hide)
     )
@@
       (effects (font (size 1.27 1.27)) (justify left))
     )
-    (property "Footprint" "" (at 196.596 91.694 90)
+    (property "Footprint" "Resistor_SMD:R_0805_2012Metric_Pad1.20x1.40mm_HandSolder" (at 196.596 91.694 90)
       (effects (font (size 1.27 1.27)) hide)
     )
@@
       (effects (font (size 1.27 1.27)) (justify left))
     )
-    (property "Footprint" "" (at 128.27 57.15 0)
+    (property "Footprint" "Capacitor_SMD:CP_Elec_8x10" (at 128.27 57.15 0)
       (effects (font (size 1.27 1.27)) hide)
     )
@@
       (effects (font (size 1.27 1.27)) (justify right))
     )
-    (property "Footprint" "" (at 60.96 93.98 0)
+    (property "Footprint" "Jumper:SolderJumper-2_P1.3mm_Bridged_Pad1.0x1.5mm" (at 60.96 93.98 0)
       (effects (font (size 1.27 1.27)) hide)
     )
@@
       (effects (font (size 1.27 1.27)))
     )
-    (property "Value" "3.9k" (at 132.08 80.01 90)
-      (effects (font (size 1.27 1.27)))
-    )
-    (property "Footprint" "" (at 132.334 82.804 90)
+    (property "Value" "2.7k" (at 132.08 80.01 90)
+      (effects (font (size 1.27 1.27)))
+    )
+    (property "Footprint" "Resistor_SMD:R_0805_2012Metric_Pad1.20x1.40mm_HandSolder" (at 132.334 82.804 90)
       (effects (font (size 1.27 1.27)) hide)
     )
@@
       (effects (font (size 1.27 1.27)) (justify left))
     )
-    (property "Footprint" "" (at 141.9352 60.96 0)
+    (property "Footprint" "Capacitor_SMD:C_0805_2012Metric_Pad1.18x1.45mm_HandSolder" (at 141.9352 60.96 0)
       (effects (font (size 1.27 1.27)) hide)
     )
@@
       (effects (font (size 1.27 1.27)) (justify left))
     )
-    (property "Footprint" "" (at 122.8852 95.25 0)
+    (property "Footprint" "Capacitor_SMD:C_0805_2012Metric_Pad1.18x1.45mm_HandSolder" (at 122.8852 95.25 0)
       (effects (font (size 1.27 1.27)) hide)
     )
@@
       (effects (font (size 1.27 1.27)) (justify left))
     )
-    (property "Footprint" "" (at 87.63 59.69 0)
-      (effects (font (size 1.27 1.27)) hide)
-    )
+    (property "Footprint" "Capacitor_SMD:CP_Elec_8x10" (at 87.63 59.69 0)
+      (effects (font (size 1.27 1.27)) hide)
+    )

Commit message: Docs
Parts:
- added C10: 10u (Optional DC Block), Capacitor_THT:CP_Radial_D5.0mm_P2.50mm, symbol Device:C_Polarized_Small_US
- C1, C9: footprint Capacitor_SMD:CP_Elec_8x10 -> Capacitor_SMD:CP_Elec_5x5.3
- RV1: footprint (none) -> Potentiometer_SMD:Potentiometer_Bourns_3314S_Horizontal
- T1: footprint (none) -> Capacitor_SMD:CP_Elec_5x5.3
- TP1: footprint (none) -> TestPoint:TestPoint_Pad_2.5x2.5mm
- U1: footprint (none) -> Package_TO_SOT_SMD:SOT-23-5_HandSoldering
Connections:
- net RIG_AF_OUT: now also C10.1; no longer T1.4 (SB)
- new net: C10.2, T1.4 (SB)
Changed lines of the file:
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@@
+    (stroke (width 0) (type default))
+  )
+  (wire (pts (xy 241.3 102.87) (xy 243.84 102.87))
     (stroke (width 0) (type default))
   )
@@
   )
   (wire (pts (xy 80.01 71.12) (xy 80.01 76.2))
-    (stroke (width 0) (type default))
-  )
-  (wire (pts (xy 236.22 102.87) (xy 243.84 102.87))
     (stroke (width 0) (type default))
   )
@@
       (effects (font (size 1.27 1.27)))
     )
-    (property "Footprint" "" (at 153.67 86.36 0)
+    (property "Footprint" "Package_TO_SOT_SMD:SOT-23-5_HandSoldering" (at 153.67 86.36 0)
       (effects (font (size 1.27 1.27)) (justify left) hide)
     )
@@
       (effects (font (size 1.27 1.27)) (justify left))
     )
-    (property "Footprint" "" (at 171.45 62.23 0)
+    (property "Footprint" "TestPoint:TestPoint_Pad_2.5x2.5mm" (at 171.45 62.23 0)
       (effects (font (size 1.27 1.27)) hide)
     )
@@
       (effects (font (size 1.27 1.27)) (justify right))
     )
-    (property "Footprint" "" (at 195.58 102.87 0)
+    (property "Footprint" "Potentiometer_SMD:Potentiometer_Bourns_3314S_Horizontal" (at 195.58 102.87 0)
       (effects (font (size 1.27 1.27)) hide)
     )
@@
       (effects (font (size 1.27 1.27)) (justify left))
     )
-    (property "Footprint" "Capacitor_SMD:CP_Elec_8x10" (at 128.27 57.15 0)
+    (property "Footprint" "Capacitor_SMD:CP_Elec_5x5.3" (at 128.27 57.15 0)
       (effects (font (size 1.27 1.27)) hide)
     )
@@
   (symbol (lib_id "Device:Transformer_1P_1S") (at 226.06 107.95 0) (unit 1)
     (in_bom yes) (on_board yes) (dnp no) (fields_autoplaced)
-    (property "Reference" "T1" (at 226.0727 97.79 0)
+    (property "Reference" "T1" (at 226.0727 100.33 0)
       (effects (font (size 1.27 1.27)))
     )
     (property "Value" "Transformer_1P_1S" (at 226.0727 100.33 0)
-      (effects (font (size 1.27 1.27)))
-    )
-    (property "Footprint" "" (at 226.06 107.95 0)
+      (effects (font (size 1.27 1.27)) hide)
+    )
+    (property "Footprint" "Capacitor_SMD:CP_Elec_5x5.3" (at 226.06 107.95 0)
       (effects (font (size 1.27 1.27)) hide)
     )
@@
     )
   )
+  (symbol (lib_id "Device:C_Polarized_Small_US") (at 238.76 102.87 270) (unit 1)
+    (in_bom yes) (on_board yes) (dnp no) (fields_autoplaced)
+    (property "Reference" "C10" (at 239.1918 96.52 90)
+      (effects (font (size 1.27 1.27)))
+    )
+    (property "Value" "10u (Optional DC Block)" (at 239.1918 99.06 90)
+      (effects (font (size 1.27 1.27)))
+    )
+    (property "Footprint" "Capacitor_THT:CP_Radial_D5.0mm_P2.50mm" (at 238.76 102.87 0)
+      (effects (font (size 1.27 1.27)) hide)
+    )
+    (property "Datasheet" "~" (at 238.76 102.87 0)
+      (effects (font (size 1.27 1.27)) hide)
+    )
+    (pin "2")
+    (pin "1")
+    (instances
+      (project "ML0"
+        (path "/5f8f636b-fd0e-498e-8696-0a023acb4c09/5945a24a-f13f-441c-8c0c-8b25494f737c"
+          (reference "C10") (unit 1)
+        )
+      )
+    )
+  )
   (symbol (lib_id "Device:C") (at 121.92 91.44 0) (unit 1)
     (in_bom yes) (on_board yes) (dnp no) (fields_autoplaced)
@@
       (effects (font (size 1.27 1.27)) (justify left))
     )
-    (property "Footprint" "Capacitor_SMD:CP_Elec_8x10" (at 87.63 59.69 0)
-      (effects (font (size 1.27 1.27)) hide)
-    )
+    (property "Footprint" "Capacitor_SMD:CP_Elec_5x5.3" (at 87.63 59.69 0)
+      (effects (font (size 1.27 1.27)) hide)
+    )

Commit message: Initial layout done
Parts:
- added R19: 1k, Resistor_SMD:R_0805_2012Metric_Pad1.20x1.40mm_HandSolder, symbol Device:R_US
- added R20: 570, Resistor_SMD:R_0805_2012Metric_Pad1.20x1.40mm_HandSolder, symbol Device:R_US
- C1: value 470u -> 100u; footprint Capacitor_SMD:CP_Elec_5x5.3 -> KiCad-Library:CAP_KEMET_530_530
- C10: value 10u (Optional DC Block) -> 47u (Optional DC Block)
- C6: value 4.7u -> 100u; footprint Capacitor_SMD:CP_Elec_8x10 -> KiCad-Library:CAP_KEMET_530_530
- C9: footprint Capacitor_SMD:CP_Elec_5x5.3 -> KiCad-Library:CAP_KEMET_530_530
- R3: value 10k -> 1k
- T1: footprint Capacitor_SMD:CP_Elec_5x5.3 -> KiCad-Library:CheapAudioTransformer
Connections:
- net GNDA: no longer RV1.3
- net RIG_GND: now also RV1.3, R20.2
- net at C6.2: now also R19.1; no longer R3.1
- net at T1.1 (AA): now also R19.2; no longer RV1.2
- net at T1.4 (SB): now also R3.1, R20.1; no longer C10.2
- net RIG_AF_OUT renamed RIG_AF_IN
- new net: C10.2, RV1.2
Other:
- moved on the sheet: C10, R3, RV1, T1

Commit message: Improvements to board
Connections:
- net RIG_GND: now also T1.4 (SB); no longer T1.3 (SA)
- net at R20.1, R3.1: now also T1.3 (SA); no longer T1.4 (SB)
Changed lines of the file:
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@@
   (junction (at 139.7 83.82) (diameter 0) (color 0 0 0 0)
   )
-  (junction (at 218.44 86.36) (diameter 0) (color 0 0 0 0)
+  (junction (at 60.96 86.36) (diameter 0) (color 0 0 0 0)
   )
-  (junction (at 60.96 86.36) (diameter 0) (color 0 0 0 0)
+  (junction (at 218.44 97.79) (diameter 0) (color 0 0 0 0)
   )
   (junction (at 128.27 50.8) (diameter 0) (color 0 0 0 0)
@@
   (junction (at 80.01 71.12) (diameter 0) (color 0 0 0 0)
   )
+  (junction (at 218.44 86.36) (diameter 0) (color 0 0 0 0)
+  )
   (junction (at 121.92 83.82) (diameter 0) (color 0 0 0 0)
-  )
-  (junction (at 218.44 96.52) (diameter 0) (color 0 0 0 0)
   )
   (junction (at 87.63 54.61) (diameter 0) (color 0 0 0 0)
@@
     (stroke (width 0) (type default))
   )
-  (wire (pts (xy 218.44 96.52) (xy 218.44 95.25))
+  (wire (pts (xy 218.44 95.25) (xy 218.44 97.79))
     (stroke (width 0) (type default))
   )
@@
   )
   (wire (pts (xy 121.92 83.82) (xy 121.92 87.63))
+    (stroke (width 0) (type default))
+  )
+  (wire (pts (xy 213.36 97.79) (xy 218.44 97.79))
     (stroke (width 0) (type default))
   )
@@
     (stroke (width 0) (type default))
   )
+  (wire (pts (xy 215.9 86.36) (xy 218.44 86.36))
+    (stroke (width 0) (type default))
+  )
   (wire (pts (xy 166.37 86.36) (xy 175.26 86.36))
     (stroke (width 0) (type default))
   )
   (wire (pts (xy 80.01 54.61) (xy 80.01 71.12))
+    (stroke (width 0) (type default))
+  )
+  (wire (pts (xy 215.9 91.44) (xy 215.9 86.36))
     (stroke (width 0) (type default))
   )
@@
     (stroke (width 0) (type default))
   )
+  (wire (pts (xy 212.09 86.36) (xy 213.36 86.36))
+    (stroke (width 0) (type default))
+  )
   (wire (pts (xy 219.71 143.51) (xy 217.17 143.51))
     (stroke (width 0) (type default))
   )
-  (wire (pts (xy 38.1 81.28) (xy 46.99 81.28))
+  (wire (pts (xy 212.09 91.44) (xy 215.9 91.44))
     (stroke (width 0) (type default))
   )
-  (wire (pts (xy 212.09 86.36) (xy 218.44 86.36))
+  (wire (pts (xy 38.1 81.28) (xy 46.99 81.28))
     (stroke (width 0) (type default))
   )
@@
     (stroke (width 0) (type default))
   )
-  (wire (pts (xy 212.09 96.52) (xy 218.44 96.52))
+  (wire (pts (xy 213.36 86.36) (xy 213.36 97.79))
     (stroke (width 0) (type default))
   )
@@
     (stroke (width 0) (type default))
   )
+  (wire (pts (xy 218.44 97.79) (xy 218.44 115.57))
+    (stroke (width 0) (type default))
+  )
   (wire (pts (xy 121.92 83.82) (xy 128.27 83.82))
     (stroke (width 0) (type default))
@@
     (stroke (width 0) (type default))
   )
+  (wire (pts (xy 212.09 96.52) (xy 212.09 91.44))
+    (stroke (width 0) (type default))
+  )
   (wire (pts (xy 50.8 83.82) (xy 57.15 83.82))
     (stroke (width 0) (type default))
   )
-  (wire (pts (xy 218.44 96.52) (xy 218.44 115.57))
-    (stroke (width 0) (type default))
-  )

Commit message: Board sent to JLC on 2024-02-26 09:18 EST
Parts:
- RV1: footprint Potentiometer_SMD:Potentiometer_Bourns_3314S_Horizontal -> KiCad-Library:POT_3362P
Changed lines of the file:
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@@
       (effects (font (size 1.27 1.27)) (justify right))
     )
-    (property "Footprint" "Potentiometer_SMD:Potentiometer_Bourns_3314S_Horizontal" (at 232.41 104.14 0)
+    (property "Footprint" "KiCad-Library:POT_3362P" (at 232.41 104.14 0)
       (effects (font (size 1.27 1.27)) hide)
     )

Commit message: First board
Other:
- note added: "BE CAREFUL WHEN ORDERING: There are different part numbers for different I2C addresses. We are using the 0 part."
Changed lines of the file:
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@@
     (effects (font (size 1.27 1.27)) (justify left bottom))
+  )
+  (text "BE CAREFUL WHEN ORDERING: There are \ndifferent part numbers for different \nI2C addresses. We are using the 0 part."
+    (at 67.31 105.41 0)
+    (effects (font (size 1.27 1.27) (color 255 12 8 1)) (justify left bottom))
   )
   (text "Attenuate line output\nto microphone level." (at 224.79 83.82 0)
