File: hw/ML1/untitled.kicad_sch (KiCad schematic)
At the start: 9 parts, among them J3 Conn_01x20, Q1 DMG2305UX-13, U7 LM4040DBZ-3

Commit message: Re-work of ML1 board in process
Parts:
- added JP2: Jumper_2_Bridged, Connector_PinHeader_2.54mm:PinHeader_1x02_P2.54mm_Vertical, symbol Jumper:Jumper_2_Bridged
- Q1: footprint digikey-footprints:SOT-23-3 -> Package_TO_SOT_SMD:SOT-23-3
- S1: footprint KiCad-Library:RPi_PicoW_SMD_TH -> bruce-footprints:RPi_PicoW_SMD_TH
Connections:
- net at S1.39 (VSYS): now also JP2.1 (A); no longer Q1.2 (S)
- net +3.3VA renamed +3.3V
- net GPIO_PWR: no longer names the net of S1.26 (GP20)
- new net: JP2.2 (B), Q1.2 (S)
- no-connect marks 5 -> 6
Other:
- note added: "Allows the Pico to be disconnected from the board power."
Changed lines of the file:
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@@
   (no_connect (at 140.97 71.12))
   (no_connect (at 140.97 111.76))
+  (no_connect (at 140.97 99.06))
   (wire (pts (xy 90.17 81.28) (xy 74.93 81.28))
     (stroke (width 0) (type default))
@@
     (stroke (width 0) (type default))
   )
+  (wire (pts (xy 162.56 64.77) (xy 162.56 68.58))
+    (stroke (width 0) (type default))
+  )
   (wire (pts (xy 88.9 106.68) (xy 88.9 114.3))
     (stroke (width 0) (type default))
@@
     (stroke (width 0) (type default))
   )
+  (wire (pts (xy 162.56 50.8) (xy 162.56 54.61))
+    (stroke (width 0) (type default))
+  )
   (wire (pts (xy 90.17 104.14) (xy 82.55 104.14))
     (stroke (width 0) (type default))
@@
     (stroke (width 0) (type default))
   )
-  (wire (pts (xy 140.97 99.06) (xy 148.59 99.06))
-    (stroke (width 0) (type default))
-  )
   (wire (pts (xy 90.17 91.44) (xy 82.55 91.44))
     (stroke (width 0) (type default))
@@
     (stroke (width 0) (type default))
   )
-  (wire (pts (xy 162.56 50.8) (xy 162.56 68.58))
-    (stroke (width 0) (type default))
-  )
   (wire (pts (xy 82.55 111.76) (xy 59.69 111.76))
     (stroke (width 0) (type default))
@@
   (wire (pts (xy 83.82 119.38) (xy 73.66 119.38))
     (stroke (width 0) (type default))
+  )
+  (text "Allows the Pico to be \ndisconnected from the \nboard power.\n"
+    (at 138.43 58.42 0)
+    (effects (font (size 1.27 1.27)) (justify left bottom))
   )
   (global_label "LED0" (shape input) (at 213.36 104.14 90) (fields_autoplaced)
@@
     )
   )
-  (global_label "GPIO_PWR" (shape input) (at 148.59 99.06 0) (fields_autoplaced)
-    (effects (font (size 1.27 1.27)) (justify left))
-    (property "Intersheetrefs" "${INTERSHEET_REFS}" (at 161.0095 99.06 0)
-      (effects (font (size 1.27 1.27)) (justify left) hide)
-    )
-  )
   (global_label "GPIO_PTT" (shape input) (at 148.59 93.98 0) (fields_autoplaced)
     (effects (font (size 1.27 1.27)) (justify left))
@@
     )
   )
+  (netclass_flag "" (length 2.54) (shape round) (at 160.02 91.44 0) (fields_autoplaced)
+    (effects (font (size 1.27 1.27)) (justify left bottom))
+    (property "Netclass" "Fast Signal" (at 160.7185 88.9 0)
+      (effects (font (size 1.27 1.27) italic) (justify left))
+    )
+  )
+  (netclass_flag "" (length 2.54) (shape round) (at 158.75 68.58 0) (fields_autoplaced)
+    (effects (font (size 1.27 1.27)) (justify left bottom))
+    (property "Netclass" "Power" (at 159.4485 66.04 0)
+      (effects (font (size 1.27 1.27) italic) (justify left))
+    )
+  )
+  (netclass_flag "" (length 2.54) (shape round) (at 147.32 88.9 0) (fields_autoplaced)
+    (effects (font (size 1.27 1.27)) (justify left bottom))
+    (property "Netclass" "Fast Signal" (at 148.0185 86.36 0)
+      (effects (font (size 1.27 1.27) italic) (justify left))
+    )
+  )
+  (netclass_flag "" (length 2.54) (shape round) (at 162.56 53.34 270) (fields_autoplaced)
+    (effects (font (size 1.27 1.27)) (justify right bottom))
+    (property "Netclass" "Power" (at 165.1 52.6415 90)
+      (effects (font (size 1.27 1.27) italic) (justify left))
+    )
+  )
   (symbol (lib_id "KC1FSZ-Symbols:SC0918_0_0") (at 115.57 100.33 0) (unit 1)
     (in_bom yes) (on_board yes) (dnp no) (fields_autoplaced)
@@
       (effects (font (size 1.27 1.27)))
     )
-    (property "Footprint" "KiCad-Library:RPi_PicoW_SMD_TH" (at 115.57 100.33 0)
+    (property "Footprint" "bruce-footprints:RPi_PicoW_SMD_TH" (at 115.57 100.33 0)
       (effects (font (size 1.27 1.27)) hide)
     )
@@
     )
   )
-  (symbol (lib_id "power:+3.3VA") (at 162.56 38.1 0) (unit 1)
-    (in_bom yes) (on_board yes) (dnp no) (fields_autoplaced)
-    (property "Reference" "#PWR023" (at 162.56 41.91 0)
-      (effects (font (size 1.27 1.27)) hide)
-    )
-    (property "Value" "+3.3VA" (at 162.56 33.02 0)
-      (effects (font (size 1.27 1.27)))
-    )
-    (property "Footprint" "" (at 162.56 38.1 0)
-      (effects (font (size 1.27 1.27)) hide)
-    )
-    (property "Datasheet" "" (at 162.56 38.1 0)
-      (effects (font (size 1.27 1.27)) hide)
-    )
-    (pin "1")
-    (instances
-      (project "ML1"
-        (path "/5f8f636b-fd0e-498e-8696-0a023acb4c09/fa333dda-eb84-4ed5-ba74-283a026e08db"
-          (reference "#PWR023") (unit 1)
-        )
-      )
-    )
-  )
   (symbol (lib_id "power:GNDA") (at 213.36 120.65 0) (unit 1)
     (in_bom yes) (on_board yes) (dnp no) (fields_autoplaced)
@@
     )
   )
+  (symbol (lib_id "Jumper:Jumper_2_Bridged") (at 162.56 59.69 90) (unit 1)
+    (in_bom yes) (on_board yes) (dnp no) (fields_autoplaced)
+    (property "Reference" "JP2" (at 163.83 59.69 90)
+      (effects (font (size 1.27 1.27)) (justify right))
+    )
+    (property "Value" "Jumper_2_Bridged" (at 163.83 60.96 90)
+      (effects (font (size 1.27 1.27)) (justify right) hide)
+    )
+    (property "Footprint" "Connector_PinHeader_2.54mm:PinHeader_1x02_P2.54mm_Vertical" (at 162.56 59.69 0)
+      (effects (font (size 1.27 1.27)) hide)
+    )
+    (property "Datasheet" "~" (at 162.56 59.69 0)
+      (effects (font (size 1.27 1.27)) hide)
+    )
+    (pin "2")
+    (pin "1")
+    (instances
+      (project "ML1"
+        (path "/5f8f636b-fd0e-498e-8696-0a023acb4c09/fa333dda-eb84-4ed5-ba74-283a026e08db"
+          (reference "JP2") (unit 1)
+        )
+      )
+    )
+  )
   (symbol (lib_id "KC1FSZ-Symbols:DMG2305UX-13") (at 162.56 45.72 0) (unit 1)
     (in_bom yes) (on_board yes) (dnp no) (fields_autoplaced)
@@
       (effects (font (size 1.27 1.27)) (justify left))
     )
-    (property "Footprint" "digikey-footprints:SOT-23-3" (at 167.64 50.8 0)
+    (property "Footprint" "Package_TO_SOT_SMD:SOT-23-3" (at 167.64 50.8 0)
       (effects (font (size 1.524 1.524)) (justify left) hide)
     )
@@
         (path "/5f8f636b-fd0e-498e-8696-0a023acb4c09/fa333dda-eb84-4ed5-ba74-283a026e08db"
           (reference "Q1") (unit 1)
+        )
+      )
+    )
+  )
+  (symbol (lib_id "power:+3.3V") (at 171.45 58.42 0) (unit 1)
+    (in_bom yes) (on_board yes) (dnp no) (fields_autoplaced)
+    (property "Reference" "#PWR03" (at 171.45 62.23 0)
+      (effects (font (size 1.27 1.27)) hide)
+    )
+    (property "Value" "+3.3V" (at 171.45 53.34 0)
+      (effects (font (size 1.27 1.27)))
+    )
+    (property "Footprint" "" (at 171.45 58.42 0)
+      (effects (font (size 1.27 1.27)) hide)
+    )
+    (property "Datasheet" "" (at 171.45 58.42 0)
+      (effects (font (size 1.27 1.27)) hide)
+    )
+    (pin "1")
+    (instances
+      (project "ML1"
+        (path "/5f8f636b-fd0e-498e-8696-0a023acb4c09/fa333dda-eb84-4ed5-ba74-283a026e08db"
+          (reference "#PWR03") (unit 1)
         )
       )
@@
     )
   )
-  (symbol (lib_id "power:+3.3VA") (at 171.45 58.42 0) (unit 1)
-    (in_bom yes) (on_board yes) (dnp no) (fields_autoplaced)
-    (property "Reference" "#PWR03" (at 171.45 62.23 0)
-      (effects (font (size 1.27 1.27)) hide)
-    )
-    (property "Value" "+3.3VA" (at 171.45 53.34 0)
-      (effects (font (size 1.27 1.27)))
-    )
-    (property "Footprint" "" (at 171.45 58.42 0)
-      (effects (font (size 1.27 1.27)) hide)
-    )
-    (property "Datasheet" "" (at 171.45 58.42 0)
-      (effects (font (size 1.27 1.27)) hide)
-    )
-    (pin "1")
-    (instances
-      (project "ML1"
-        (path "/5f8f636b-fd0e-498e-8696-0a023acb4c09/fa333dda-eb84-4ed5-ba74-283a026e08db"
-          (reference "#PWR03") (unit 1)
-        )
-      )
-    )
-  )
   (symbol (lib_id "Device:R") (at 171.45 67.31 0) (unit 1)
     (in_bom yes) (on_board yes) (dnp no) (fields_autoplaced)
@@
         )
       )
+    )
+  )
+  (symbol (lib_id "power:+3.3V") (at 162.56 38.1 0) (unit 1)
+    (in_bom yes) (on_board yes) (dnp no) (fields_autoplaced)
+    (property "Reference" "#PWR023" (at 162.56 41.91 0)
+      (effects (font (size 1.27 1.27)) hide)
+    )
+    (property "Value" "+3.3V" (at 162.56 33.02 0)
+      (effects (font (size 1.27 1.27)))
+    )
+    (property "Footprint" "" (at 162.56 38.1 0)
+      (effects (font (size 1.27 1.27)) hide)
+    )
+    (property "Datasheet" "" (at 162.56 38.1 0)
+      (effects (font (size 1.27 1.27)) hide)
+    )
+    (pin "1")
+    (instances
+      (project "ML1"
+        (path "/5f8f636b-fd0e-498e-8696-0a023acb4c09/fa333dda-eb84-4ed5-ba74-283a026e08db"
+          (reference "#PWR023") (unit 1)
+        )
+      )

Commit message: Final checks, preparing to create GRB
Parts:
- Q1: symbol KC1FSZ-Symbols:DMG2305UX-13 -> symbol-library-1:DMG2305UX-13
- S1: symbol KC1FSZ-Symbols:SC0918_0_0 -> symbol-library-1:SC0918_0_0
Other:
- note added: "This is a voltage reference for the ADC"
Changed lines of the file:
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@@
+	)
+	(junction
+		(at 162.56 73.66)
+		(diameter 0)
+		(color 0 0 0 0)
 	)
 	(junction
@@
 	(wire
 		(pts
+			(xy 162.56 73.66) (xy 171.45 73.66)
+		)
+		(stroke
+			(width 0)
+			(type default)
+		)
+	)
+	(wire
+		(pts
 			(xy 87.63 109.22) (xy 87.63 116.84)
 		)
@@
 	(wire
 		(pts
-			(xy 140.97 73.66) (xy 171.45 73.66)
+			(xy 140.97 73.66) (xy 162.56 73.66)
 		)
 		(stroke
@@
 			(width 0)
 			(type default)
+		)
+	)
+	(text "This is a voltage reference for the ADC"
+		(exclude_from_sim no)
+		(at 177.546 72.136 0)
+		(effects
+			(font
+				(size 1.27 1.27)
+			)
 		)
 	)
@@
 	)
 	(symbol
-		(lib_id "KC1FSZ-Symbols:SC0918_0_0")
+		(lib_id "symbol-library-1:SC0918_0_0")
 		(at 115.57 100.33 0)
 		(unit 1)
@@
 		(fields_autoplaced yes)
 		(property "Reference" "S1"
-			(at 115.57 54.61 0)
+			(at 115.57 53.34 0)
 			(effects
 				(font
@@
 		)
 		(property "Value" "~"
-			(at 115.57 100.33 0)
+			(at 115.57 55.88 0)
 			(effects
 				(font
@@
 			)
 		)
-		(property "Description" ""
+		(property "Description" "Generic connector, single row, 01x20, script generated (kicad-library-utils/schlib/autogen/connector/)"
 			(at 54.61 96.52 0)
 			(effects
@@
 			)
 		)
-		(property "Description" ""
+		(property "Description" "Power symbol creates a global label with name \"GNDA\" , analog ground"
 			(at 213.36 120.65 0)
 			(effects
@@
 			)
 		)
-		(property "Description" ""
+		(property "Description" "Light emitting diode"
 			(at 213.36 116.84 0)
 			(effects
@@
 				(path "/5f8f636b-fd0e-498e-8696-0a023acb4c09/fa333dda-eb84-4ed5-ba74-283a026e08db"
 					(reference "D3")
+					(unit 1)
+				)
+			)
+		)
+	)
+	(symbol
+		(lib_id "power:PWR_FLAG")
+		(at 162.56 73.66 180)
+		(unit 1)
+		(exclude_from_sim no)
+		(in_bom yes)
+		(on_board yes)
+		(dnp no)
+		(fields_autoplaced yes)
+		(property "Reference" "#FLG03"
+			(at 162.56 75.565 0)
+			(effects
+				(font
+					(size 1.27 1.27)
+				)
+				(hide yes)
+			)
+		)
+		(property "Value" "PWR_FLAG"
+			(at 162.56 78.74 0)
+			(effects
+				(font
+					(size 1.27 1.27)
+				)
+			)
+		)
+		(property "Footprint" ""
+			(at 162.56 73.66 0)
+			(effects
+				(font
+					(size 1.27 1.27)
+				)
+				(hide yes)
+			)
+		)
+		(property "Datasheet" "~"
+			(at 162.56 73.66 0)
+			(effects
+				(font
+					(size 1.27 1.27)
+				)
+				(hide yes)
+			)
+		)
+		(property "Description" "Special symbol for telling ERC where power comes from"
+			(at 162.56 73.66 0)
+			(effects
+				(font
+					(size 1.27 1.27)
+				)
+				(hide yes)
+			)
+		)
+		(pin "1"
+		)
+		(instances
+			(project "ML1"
+				(path "/5f8f636b-fd0e-498e-8696-0a023acb4c09/fa333dda-eb84-4ed5-ba74-283a026e08db"
+					(reference "#FLG03")
 					(unit 1)
 				)
@@
 			)
 		)
-		(property "Description" ""
+		(property "Description" "Power symbol creates a global label with name \"GNDA\" , analog ground"
 			(at 171.45 81.28 0)
 			(effects
@@
 			)
 		)
-		(property "Description" ""
+		(property "Description" "Jumper, 2-pole, closed/bridged"
 			(at 162.56 59.69 0)
 			(effects
@@
 	)
 	(symbol
-		(lib_id "KC1FSZ-Symbols:DMG2305UX-13")
+		(lib_id "symbol-library-1:DMG2305UX-13")
 		(at 162.56 45.72 0)
 		(unit 1)
@@
 		(fields_autoplaced yes)
 		(property "Reference" "Q1"
-			(at 166.37 44.45 0)
+			(at 166.37 44.4499 0)
 			(effects
 				(font
@@
 		)
 		(property "Value" "DMG2305UX-13"
-			(at 166.37 46.99 0)
+			(at 166.37 46.9899 0)
 			(effects
 				(font
@@
 			)
 		)
-		(property "Description" ""
+		(property "Description" "Power symbol creates a global label with name \"+3.3V\""
 			(at 171.45 58.42 0)
 			(effects
@@
 			)
 		)
-		(property "Description" ""
+		(property "Description" "Resistor, small US symbol"
 			(at 227.33 110.49 0)
 			(effects
@@
 			)
 		)
-		(property "Description" ""
+		(property "Description" "Resistor, small US symbol"
 			(at 213.36 110.49 0)
 			(effects
@@
 			)
 		)
-		(property "Description" ""
+		(property "Description" "3.000V Precision Micropower Shunt Voltage Reference, SOT-23"
 			(at 171.45 77.47 0)
 			(effects
@@
 			)
 		)
-		(property "Description" ""
+		(property "Description" "Power symbol creates a global label with name \"GNDA\" , analog ground"
 			(at 227.33 120.65 0)
 			(effects
@@
 			)
 		)
-		(property "Description" ""
+		(property "Description" "Light emitting diode"
 			(at 227.33 116.84 0)
 			(effects
@@
 			)
 		)
-		(property "Description" ""
+		(property "Description" "Power symbol creates a global label with name \"GNDA\" , analog ground"
 			(at 63.5 125.73 0)
 			(effects
@@
 			)
 		)
-		(property "Description" ""
+		(property "Description" "Resistor"
 			(at 171.45 67.31 0)
 			(effects
@@
 			)
 		)
-		(property "Description" ""
+		(property "Description" "Power symbol creates a global label with name \"+3.3V\""
 			(at 162.56 38.1 0)
 			(effects
@@
 			)
 		)
-		(property "Description" ""
+		(property "Description" "Power symbol creates a global label with name \"GNDA\" , analog ground"
 			(at 85.09 142.24 0)
 			(effects

Commit message: Final checks, preparing to create GRB
Other:
- company: (none) -> Bruce MacKinnon KC1FSZ
- title: (none) -> MicroLink - Microcontroller
Changed lines of the file:
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@@
 	(generator "eeschema")
 	(generator_version "8.0")
-	(paper "A4")
+	(paper "USLetter")
+	(title_block
+		(title "MicroLink - Microcontroller")
+		(date "2024-03-28")
+		(rev "1")
+		(company "Bruce MacKinnon KC1FSZ")
+		(comment 1 "Copyright (C) 2024 - Not For Commercial Use")
+	)
 	(junction
 		(at 63.5 104.14)
