File: hw/ML2/untitled.kicad_sch (KiCad schematic)
At the start: 9 parts, among them J3 Conn_01x20, Q1 DMG2305UX-13, U7 LM4040DBZ-3

Commit message: Board passing checks, ready for review
Parts:
- added SW0: TS04-66-55-BK-160-SMT, bruce-footprints:SW_TS04-66-55-BK-160-SMT, symbol symbol-library-1:TS04-66-55-BK-160-SMT
Connections:
- net GNDA: now also SW0.2, SW0.4
- net SW0: now reaches S1.26 (GP20)
- net SW0: now also SW0.1, SW0.3
- no-connect marks 6 -> 5
