File: hw/ML2/ML2.kicad_pcb (KiCad board)
At the start: 2 copper layers, 125 x 56 mm, 72 parts, among them J1 Conn_01x07, J2 5-12V Supply, J3 Conn_01x20, J4 Conn_01x02, Q1 DMG2305UX-13, T1 Transformer_1P_1S, T2 Transformer_1P_1S, U1 LMV324 (Actually LTV9161), U2 LTV-356T, U3 NCP1117-3.3_SOT223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

Commit message: Board passing checks, ready for review
Parts:
- added SW0: TS04-66-55-BK-160-SMT, bruce-footprints:SW_TS04-66-55-BK-160-SMT, F.Cu at (170.0, 81.5)
- moved H2 0.18 mm to (239.8, 47.0)
- moved H3 0.13 mm to (121.7, 47.0)
Connections:
- S1 pad 26: unconnected-(S1-GP20-Pad26)_0 -> SW0
Routing:
- net SW0: track 0.00 -> 24.5 mm
- net GNDA: track 32.5 -> 27.8 mm, vias 127 -> 135
Other:
- outline, holes or cut-outs redrawn
- board text added: "Cleared for WIFI Antenna and SWD pins."

Commit message: Plot files generated for fab
Routing:
- net GNDA: vias 135 -> 138
Other:
- board text added: "COS"
- board text added: "IN"
- board text added: "O+"
- board text added: "O-"
- board text added: "PTT"
- board text removed: "Radio"
Changed lines of the file:
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@@
+		)
+	)
+	(gr_text "COS"
+		(at 238.506 58.928 0)
+		(layer "F.SilkS")
+		(effects
+			(font
+				(size 1 1)
+				(thickness 0.15)
+			)
+			(justify left bottom)
 		)
 	)
@@
 		)
 	)
+	(gr_text "O-"
+		(at 238.506 56.134 0)
+		(layer "F.SilkS")
+		(effects
+			(font
+				(size 1 1)
+				(thickness 0.15)
+			)
+			(justify left bottom)
+		)
+	)
 	(gr_text "GND"
 		(at 122.936 77.216 0)
@@
 		)
 	)
+	(gr_text "IN"
+		(at 238.506 66.294 0)
+		(layer "F.SilkS")
+		(effects
+			(font
+				(size 1 1)
+				(thickness 0.15)
+			)
+			(justify left bottom)
+		)
+	)
 	(gr_text "LED0"
 		(at 163.068 80.518 0)
@@
 		)
 	)
+	(gr_text "PTT"
+		(at 238.506 64.008 0)
+		(layer "F.SilkS")
+		(effects
+			(font
+				(size 1 1)
+				(thickness 0.15)
+			)
+			(justify left bottom)
+		)
+	)
 	(gr_text "1"
-		(at 239.168 54.356 0)
+		(at 237.744 51.816 0)
 		(layer "F.SilkS")
 		(effects
@@
 		)
 	)
-	(gr_text "Radio"
-		(at 240.692 62.738 90)
+	(gr_text "GND"
+		(at 238.506 61.214 0)
 		(layer "F.SilkS")
 		(effects
 			(font
-				(size 1.5 1.5)
-				(thickness 0.3)
-				(bold yes)
+				(size 1 1)
+				(thickness 0.15)
 			)
 			(justify left bottom)
@@
 		)
 	)
+	(gr_text "GND"
+		(at 238.506 68.834 0)
+		(layer "F.SilkS")
+		(effects
+			(font
+				(size 1 1)
+				(thickness 0.15)
+			)
+			(justify left bottom)
+		)
+	)
+	(gr_text "O+"
+		(at 238.506 53.594 0)
+		(layer "F.SilkS")
+		(effects
+			(font
+				(size 1 1)
+				(thickness 0.15)
+			)
+			(justify left bottom)
+		)
+	)
 	(gr_text "Cleared for WIFI \nAntenna and SWD\npins."
 		(at 145.542 85.598 0)
@@
 	)
 	(via
+		(at 164.338 87.122)
+		(size 0.8)
+		(drill 0.4)
+		(layers "F.Cu" "B.Cu")
+		(free yes)
+		(net 2)
+	)
+	(via
 		(at 131.826 97.79)
 		(size 0.8)
@@
 	)
 	(via
+		(at 162.052 84.836)
+		(size 0.8)
+		(drill 0.4)
+		(layers "F.Cu" "B.Cu")
+		(free yes)
+		(net 2)
+	)
+	(via
 		(at 217.424 65.278)
 		(size 0.8)
@@
 	(via
 		(at 173.99 80.264)
+		(size 0.8)
+		(drill 0.4)
+		(layers "F.Cu" "B.Cu")
+		(free yes)
+		(net 2)
+	)
+	(via
+		(at 166.878 89.662)
 		(size 0.8)
 		(drill 0.4)
@@
 	)
 	(via
-		(at 240.03 64.008)
+		(at 240.03 61.976)
 		(size 0.8)
 		(drill 0.4)
@@
 	)
 	(via
-		(at 240.03 55.372)
-		(size 0.8)
-		(drill 0.4)
+		(at 240.03 56.896)
+		(size 0.8)
+		(drill 0.4)
