File: hw/ML3/untitled.kicad_sch (KiCad schematic)
At the start: 10 parts, among them J3 Conn_01x20, Q1 DMG2305UX-13, SW0 TS04-66-55-BK-160-SMT, U7 LM4040DBZ-3

Commit message: ML3 board modified for improved case/DFM.  Sending this version to Steve
Parts:
- removed JP2: Jumper_2_Bridged, Connector_PinHeader_2.54mm:PinHeader_1x02_P2.54mm_Vertical, symbol Jumper:Jumper_2_Bridged
- added JP1: SolderJumper_2_Bridged, Jumper:SolderJumper-2_P1.3mm_Bridged_Pad1.0x1.5mm, symbol Jumper:SolderJumper_2_Bridged
Connections:
- net at S1.39 (VSYS): now also JP1.1 (A)
- net at Q1.2 (S): now also JP1.2 (B)
Changed lines of the file:
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@@
 	(title_block
 		(title "MicroLink - Microcontroller")
-		(date "2024-04-10")
-		(rev "2")
+		(date "2024-04-15")
+		(rev "3")
 		(company "Bruce MacKinnon KC1FSZ")
 		(comment 1 "Copyright (C) 2024 - Not For Commercial Use")
@@
 	(wire
 		(pts
-			(xy 162.56 64.77) (xy 162.56 68.58)
+			(xy 162.56 62.23) (xy 162.56 68.58)
 		)
 		(stroke
@@
 	(text "Allows the Pico to be \ndisconnected from the \nboard power.\n"
 		(exclude_from_sim no)
-		(at 138.43 58.42 0)
+		(at 173.228 57.912 0)
 		(effects
 			(font
@@
 		)
 		(instances
-			(project "ML2"
+			(project "ML3"
 				(path "/5f8f636b-fd0e-498e-8696-0a023acb4c09/fa333dda-eb84-4ed5-ba74-283a026e08db"
 					(reference "SW0")
@@
 		)
 		(instances
-			(project "ML2"
+			(project "ML3"
 				(path "/5f8f636b-fd0e-498e-8696-0a023acb4c09/fa333dda-eb84-4ed5-ba74-283a026e08db"
 					(reference "S1")
@@
 		)
 		(instances
-			(project "ML2"
+			(project "ML3"
 				(path "/5f8f636b-fd0e-498e-8696-0a023acb4c09/fa333dda-eb84-4ed5-ba74-283a026e08db"
 					(reference "J3")
@@
 		)
 		(instances
-			(project "ML2"
+			(project "ML3"
 				(path "/5f8f636b-fd0e-498e-8696-0a023acb4c09/fa333dda-eb84-4ed5-ba74-283a026e08db"
 					(reference "#PWR043")
@@
 		)
 		(instances
-			(project "ML2"
+			(project "ML3"
 				(path "/5f8f636b-fd0e-498e-8696-0a023acb4c09/fa333dda-eb84-4ed5-ba74-283a026e08db"
 					(reference "D3")
@@
 		)
 		(instances
-			(project "ML2"
+			(project "ML3"
 				(path "/5f8f636b-fd0e-498e-8696-0a023acb4c09/fa333dda-eb84-4ed5-ba74-283a026e08db"
 					(reference "#PWR029")
@@
 		)
 		(instances
-			(project "ML2"
+			(project "ML3"
 				(path "/5f8f636b-fd0e-498e-8696-0a023acb4c09/fa333dda-eb84-4ed5-ba74-283a026e08db"
 					(reference "#FLG03")
@@
 		)
 		(instances
-			(project "ML2"
+			(project "ML3"
 				(path "/5f8f636b-fd0e-498e-8696-0a023acb4c09/fa333dda-eb84-4ed5-ba74-283a026e08db"
 					(reference "#PWR022")
-					(unit 1)
-				)
-			)
-		)
-	)
-	(symbol
-		(lib_id "Jumper:Jumper_2_Bridged")
-		(at 162.56 59.69 90)
-		(unit 1)
-		(exclude_from_sim no)
-		(in_bom yes)
-		(on_board yes)
-		(dnp no)
-		(fields_autoplaced yes)
-		(property "Reference" "JP2"
-			(at 163.83 59.69 90)
-			(effects
-				(font
-					(size 1.27 1.27)
-				)
-				(justify right)
-			)
-		)
-		(property "Value" "Jumper_2_Bridged"
-			(at 163.83 60.96 90)
-			(effects
-				(font
-					(size 1.27 1.27)
-				)
-				(justify right)
-				(hide yes)
-			)
-		)
-		(property "Footprint" "Connector_PinHeader_2.54mm:PinHeader_1x02_P2.54mm_Vertical"
-			(at 162.56 59.69 0)
-			(effects
-				(font
-					(size 1.27 1.27)
-				)
-				(hide yes)
-			)
-		)
-		(property "Datasheet" "~"
-			(at 162.56 59.69 0)
-			(effects
-				(font
-					(size 1.27 1.27)
-				)
-				(hide yes)
-			)
-		)
-		(property "Description" "Jumper, 2-pole, closed/bridged"
-			(at 162.56 59.69 0)
-			(effects
-				(font
-					(size 1.27 1.27)
-				)
-				(hide yes)
-			)
-		)
-		(pin "2"
-		)
-		(pin "1"
-		)
-		(instances
-			(project "ML2"
-				(path "/5f8f636b-fd0e-498e-8696-0a023acb4c09/fa333dda-eb84-4ed5-ba74-283a026e08db"
-					(reference "JP2")
 					(unit 1)
 				)
@@
 		)
 		(instances
-			(project "ML2"
+			(project "ML3"
 				(path "/5f8f636b-fd0e-498e-8696-0a023acb4c09/fa333dda-eb84-4ed5-ba74-283a026e08db"
 					(reference "Q1")
@@
 		)
 		(instances
-			(project "ML2"
+			(project "ML3"
 				(path "/5f8f636b-fd0e-498e-8696-0a023acb4c09/fa333dda-eb84-4ed5-ba74-283a026e08db"
 					(reference "R20")
@@
 		)
 		(instances
-			(project "ML2"
+			(project "ML3"
 				(path "/5f8f636b-fd0e-498e-8696-0a023acb4c09/fa333dda-eb84-4ed5-ba74-283a026e08db"
 					(reference "R17")
@@
 		)
 		(instances
-			(project "ML2"
+			(project "ML3"
 				(path "/5f8f636b-fd0e-498e-8696-0a023acb4c09/fa333dda-eb84-4ed5-ba74-283a026e08db"
 					(reference "U7")
+					(unit 1)
+				)
+			)
+		)
+	)
+	(symbol
+		(lib_id "Jumper:SolderJumper_2_Bridged")
+		(at 162.56 58.42 90)
+		(unit 1)
+		(exclude_from_sim yes)
+		(in_bom no)
+		(on_board yes)
+		(dnp no)
+		(fields_autoplaced yes)
+		(property "Reference" "JP1"
+			(at 165.1 57.1499 90)
+			(effects
+				(font
+					(size 1.27 1.27)
+				)
+				(justify right)
+			)
+		)
+		(property "Value" "SolderJumper_2_Bridged"
+			(at 165.1 59.6899 90)
+			(effects
+				(font
+					(size 1.27 1.27)
+				)
+				(justify right)
+			)
+		)
+		(property "Footprint" "Jumper:SolderJumper-2_P1.3mm_Bridged_Pad1.0x1.5mm"
+			(at 162.56 58.42 0)
+			(effects
+				(font
+					(size 1.27 1.27)
+				)
+				(hide yes)
+			)
+		)
+		(property "Datasheet" "~"
+			(at 162.56 58.42 0)
+			(effects
+				(font
+					(size 1.27 1.27)
+				)
+				(hide yes)
+			)
+		)
+		(property "Description" "Solder Jumper, 2-pole, closed/bridged"
+			(at 162.56 58.42 0)
+			(effects
+				(font
+					(size 1.27 1.27)
+				)
+				(hide yes)
+			)
+		)
+		(pin "1"
+		)
+		(pin "2"
+		)
+		(instances
+			(project "ML3"
+				(path "/5f8f636b-fd0e-498e-8696-0a023acb4c09/fa333dda-eb84-4ed5-ba74-283a026e08db"
+					(reference "JP1")
 					(unit 1)
 				)
@@
 		)
 		(instances
-			(project "ML2"
+			(project "ML3"
 				(path "/5f8f636b-fd0e-498e-8696-0a023acb4c09/fa333dda-eb84-4ed5-ba74-283a026e08db"
 					(reference "#PWR045")
@@
 		)
 		(instances
-			(project "ML2"
+			(project "ML3"
 				(path "/5f8f636b-fd0e-498e-8696-0a023acb4c09/fa333dda-eb84-4ed5-ba74-283a026e08db"
 					(reference "D4")
@@
 		)
 		(instances
-			(project "ML2"
+			(project "ML3"
 				(path "/5f8f636b-fd0e-498e-8696-0a023acb4c09/fa333dda-eb84-4ed5-ba74-283a026e08db"
 					(reference "#PWR06")
@@
 		)
 		(instances
-			(project "ML2"
+			(project "ML3"
 				(path "/5f8f636b-fd0e-498e-8696-0a023acb4c09/fa333dda-eb84-4ed5-ba74-283a026e08db"
 					(reference "#PWR023")
@@
 		)
 		(instances
-			(project "ML2"
+			(project "ML3"
 				(path "/5f8f636b-fd0e-498e-8696-0a023acb4c09/fa333dda-eb84-4ed5-ba74-283a026e08db"
 					(reference "#PWR027")
