File: hw/ML4/Power.kicad_sch (KiCad schematic)
At the start: 10 parts, among them J4 Conn_01x02, U3 NCP1117-3.3_SOT223

Commit message: Updates for ML4
Parts:
- R22: value 220 -> 100
Changed lines of the file:
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@@
 			)
 		)
-		(property "Value" "220"
+		(property "Value" "100"
 			(at 205.74 82.55 0)
 			(effects

Commit message: Working on JCSC BOM
Parts:
- R21: LCSC (none) -> C17675
- R22: LCSC (none) -> C17408

Commit message: Working on adding LCSC part numbers
Parts:
- removed C1, C2: 10u, bruce-footprints:CPOL_0805_2012Metric_Pad1.18x1.45mm_HandSolder, symbol Device:C_Polarized_Small_US
- removed C8, C9: 47u, bruce-footprints:CPOL_0805_2012Metric_Pad1.18x1.45mm_HandSolder, symbol Device:C_Polarized_Small_US
- removed U3: NCP1117-3.3_SOT223, Package_TO_SOT_SMD:SOT-223-3_TabPin2, symbol Regulator_Linear:NCP1117-3.3_SOT223
- added C1, C2: 22u, Capacitor_SMD:C_0805_2012Metric_Pad1.18x1.45mm_HandSolder, symbol Device:C_Small
- added C8, C9: 47u, Capacitor_SMD:C_0805_2012Metric_Pad1.18x1.45mm_HandSolder, symbol Device:C_Small
- added R7: 10, Resistor_SMD:R_0805_2012Metric_Pad1.20x1.40mm_HandSolder, symbol Device:R_US
- added U3: LM1117MP-3.3, Package_TO_SOT_SMD:SOT-223-3_TabPin2, symbol Regulator_Linear:LM1117MP-3.3
- D1: LCSC (none) -> C84256
Connections:
- net +3.3V: now also R7.1, U3.2 (VO)
- net +3.3VA: now also C8.1, C9.1
- net GNDA: now also C1.2, C2.2, C8.2, C9.2, U3.1 (GND)
- new net: C2.1, R7.2
- new net +12VA: C1.1, U3.3 (VI)
Other:
- note added: "Per datasheet: "output capacitor minimum of 4.7uF with ESR in range of 33mO to 2.2O for stability." The ESR for a ceramic is too small, so added series R."
- note added: "Watch out, must be +12V capable!"
- note removed: "Per datasheet: "output capacitor minimum of 4.7uF with ESR in range of 33mO to 2.2O" Using tanalum."

Commit message: Working on adding LCSC part numbers
Parts:
- U3: LCSC C9662 -> C9662
Changed lines of the file:
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@@
 			)
 		)
-		(property "LCSC" " C9662"
+		(property "LCSC" "C9662"
 			(at 80.01 80.01 0)
 			(effects
@@
 					(size 1.27 1.27)
 				)
+				(hide yes)
 			)
 		)
@@
 					(size 1.27 1.27)
 				)
-			)
-		)
+				(hide yes)
+			)
+		)
+		(property "Sim.Pins" "1=K 2=A"
+			(at 203.2 87.63 0)
+			(effects
+				(font
+					(size 1.27 1.27)
+				)
+				(hide yes)
+			)
+		)

Commit message: Working on adding LCSC part numbers
Parts:
- J4: BOM Comments (none) -> Standard 2.54mm pin header; LCSC (none) -> C492401
- TP5: BOM Comments (none) -> No component, PCB test point; now left out of the parts list
Changed lines of the file:
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@@
 			)
 		)
-		(property "LCSC" ""
+		(property "LCSC" "C492401"
 			(at 129.54 127 0)
 			(effects
@@
 					(size 1.27 1.27)
 				)
+			)
+		)
+		(property "BOM Comments" "Standard 2.54mm pin header"
+			(at 129.54 127 0)
+			(effects
+				(font
+					(size 1.27 1.27)
+				)
+				(hide yes)
 			)
 		)
@@
 		(unit 1)
 		(exclude_from_sim no)
-		(in_bom yes)
+		(in_bom no)
 		(on_board yes)
 		(dnp no)
@@
 			)
 		)
+		(property "BOM Comments" "No component, PCB test point"
+			(at 165.1 114.3 0)
+			(effects
+				(font
+					(size 1.27 1.27)
+				)
+				(hide yes)
+			)
+		)
+		(property "DK" ""
+			(at 165.1 114.3 0)
+			(effects
+				(font
+					(size 1.27 1.27)
+				)
+				(hide yes)
+			)
+		)
