File: hw/ML4/untitled.kicad_sch (KiCad schematic)
At the start: 10 parts, among them J3 Conn_01x20, Q1 DMG2305UX-13, SW0 TS04-66-55-BK-160-SMT, U7 LM4040D30IDBZR

Commit message: Working on docs
Parts:
- S1: value ~ -> Pico W Module
Changed lines of the file:
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@@
 			)
 		)
-		(property "Value" "~"
+		(property "Value" "Pico W Module"
 			(at 115.57 55.88 0)
 			(effects
