File: hw/ML4/AudioOut.kicad_sch (KiCad schematic)
At the start: 23 parts, among them U1 TLV9164PWR, U2 LTV-356T, U4 MCP4725A0T-E/CH

Commit message: Working on docs
Parts:
- R24: value 2,.2k -> 2.2k
Changed lines of the file:
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@@
 			)
 		)
-		(property "Value" "2,.2k"
+		(property "Value" "2.2k"
 			(at 227.076 94.996 0)
 			(effects
@@
 			(at 232.41 90.17 0)
 			(effects
+				(font
+					(size 1.27 1.27)
+				)
+				(hide yes)
+			)
+		)
+		(property "DK" ""
+			(at 232.41 90.17 0)
+			(effects
+				(font
+					(size 1.27 1.27)
+				)
+				(hide yes)
+			)
+		)
+		(property "BOM Comments" ""
+			(at 232.41 90.17 0)
+			(effects

Commit message: Docs
Changed lines of the file:
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@@
 		)
 		(property "Value" "47u (Optional DC Block)"
-			(at 256.54 91.44 90)
+			(at 253.238 91.44 90)
 			(effects
 				(font
