File: hw/ML4/ML4.kicad_pcb (KiCad board)
At the start: 2 copper layers, 130 x 56 mm, 73 parts, among them J1 DE9_Receptacle, J2 PJ-102AH, J3 Conn_01x20, J4 Conn_01x02, Q1 DMG2305UX-13, SW0 TS04-66-55-BK-160-SMT, T1 Transformer_1P_1S, T2 Transformer_1P_1S, U1 LMV324 (Actually LTV9161), U2 LTV-356T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

Commit message: Updates for ML4
Changed lines of the file:
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@@
 		(tags "resistor handsolder")
 		(property "Reference" "R9"
-			(at 2.032 2.794 90)
+			(at -0.112 1.766 90)
 			(layer "F.SilkS")
 			(effects
@@
 		(layer "Edge.Cuts")
 	)
+	(gr_text "+"
+		(at 126.8 78.1 0)
+		(layer "F.SilkS")
+		(effects
+			(font
+				(size 0.8 0.8)
+				(thickness 0.15)
+			)
+			(justify left bottom)
+		)
+	)
 	(gr_text "GND"
 		(at 91.436 52.07 0)
@@
 		)
 	)
+	(gr_text "+"
+		(at 158.95 46.8 0)
+		(layer "F.SilkS")
+		(effects
+			(font
+				(size 0.8 0.8)
+				(thickness 0.15)
+			)
+			(justify left bottom)
+		)
+	)
 	(gr_text "MicroLink V3\n2024-04 KC1FSZ"
 		(at 163.572 97.79 0)
@@
 		)
 	)
+	(gr_text "+"
+		(at 126.75 72.25 0)
+		(layer "F.SilkS")
+		(effects
+			(font
+				(size 0.8 0.8)
+				(thickness 0.15)
+			)
+			(justify left bottom)
+		)
+	)

Commit message: Working on JCSC BOM
Other:
- board text added: "MicroLink V4 2025-09 KC1FSZ"
- board text removed: "MicroLink V3 2024-04 KC1FSZ"

Commit message: Working on adding LCSC part numbers
Parts:
- removed R23: 0R, Resistor_SMD:R_0805_2012Metric_Pad1.20x1.40mm_HandSolder
- added R7: 10, Resistor_SMD:R_0805_2012Metric_Pad1.20x1.40mm_HandSolder, F.Cu at (139.5, 63.0)
- C1: value 10u -> 47u; footprint bruce-footprints:CPOL_0805_2012Metric_Pad1.18x1.45mm_HandSolder -> Capacitor_SMD:C_0805_2012Metric_Pad1.18x1.45mm_HandSolder
- C11, C19, C20, C5, C7, C8, C9: footprint bruce-footprints:CPOL_0805_2012Metric_Pad1.18x1.45mm_HandSolder -> Capacitor_SMD:C_0805_2012Metric_Pad1.18x1.45mm_HandSolder
- C2: value 10u -> 22u; footprint bruce-footprints:CPOL_0805_2012Metric_Pad1.18x1.45mm_HandSolder -> Capacitor_SMD:C_0805_2012Metric_Pad1.18x1.45mm_HandSolder
- R17, R20, R22: value 220 -> 100
- R24: value 1k -> 2,.2k
- R25: value 33k -> 39k
- R4: footprint Resistor_SMD:R_0805_2012Metric_Pad1.20x1.40mm_HandSolder -> Resistor_THT:R_Axial_DIN0309_L9.0mm_D3.2mm_P2.54mm_Vertical
- R5, R6: value 10k -> 2.2k
- R8: value 200 -> 220
- RV1: value 10k -> 50k
- U3: value NCP1117-3.3_SOT223 -> LM1117MP-3.3
- moved R4 8.01 mm to (202.9, 78.5), turned to -90 degrees
- moved C8 4.55 mm to (147.0, 54.0)
- moved C2 2.75 mm to (139.5, 66.0), turned to 180 degrees
- moved C9 1.30 mm to (148.0, 50.5), turned to 0 degrees
- moved R24 1.29 mm to (203.0, 86.4), turned to 90 degrees
- moved U7 0.90 mm to (128.0, 58.0)
- moved R25 0.63 mm to (199.0, 78.5)
- moved C20 0.36 mm to (159.5, 54.5)
- moved C19 0.35 mm to (176.0, 49.0)
- moved C1 0.25 mm to (139.5, 60.5)
- moved C7 0.25 mm to (167.0, 75.0)
- moved C11 0.15 mm to (167.0, 77.5)
- moved U3 0.13 mm to (132.7, 64.0)
- moved C5 0.09 mm to (147.2, 76.0)
Connections:
- C2 pad 1: +3.3V -> Net-(C2-Pad1)
- R24 pad 2: Net-(C10-Pad2) -> Net-(R24-Pad2)
- R25 pad 2: Net-(R25-Pad2) -> Net-(R24-Pad2)
- RV1 pad 1: Net-(R23-Pad2) -> RIG_GND
- RV1 pad 3: Net-(R25-Pad2) -> Net-(R24-Pad2)
Routing:
- net Net-(R24-Pad2): track 0.00 -> 20.7 mm
- net Net-(R25-Pad2): track 17.4 -> 0.00 mm
- net GNDA: track 29.6 -> 23.4 mm, vias 144 -> 141
- net +3.3VA: track 127.5 -> 132.2 mm
- net Net-(C10-Pad2): track 11.1 -> 7.76 mm
- net Net-(R23-Pad2): track 3.15 -> 0.00 mm
- net Net-(C2-Pad1): track 0.00 -> 3.08 mm
- net Net-(S1-ADC_VREF): track 5.87 -> 4.91 mm
- net Net-(T1-SA): track 12.8 -> 12.1 mm
- net RIG_GND: vias 12 -> 14

Commit message: Working on ML4
Parts:
- removed T1, T2: Transformer_1P_1S, bruce-footprints:CheapAudioTransformer
- added TR1: SM-LP-5001, bruce-footprints:TRAN6_SM-LP-5001_BRN, F.Cu at (187.8, 88.2)
- added TR2: SM-LP-5001, bruce-footprints:TRAN6_SM-LP-5001_BRN, F.Cu at (187.8, 55.3)
- C1: value 47u -> 22u
- C17: value 1u -> 47u
- Q1: footprint Package_TO_SOT_SMD:SOT-23-3 -> Package_TO_SOT_SMD:SOT-23_Handsoldering
- R26: value 0R -> 0R 1206
- R4: value 570 -> 620
- RV2: value 10k -> 50k
- U1: value LMV324 (Actually LTV9161) -> TLV9164PWR
- U4: value MCP4725xxx-xCH -> MCP4725A0T-E/CH
- U7: value LM4040DBZ-3 -> LM4040D30IDBZR
- moved Q1 0.36 mm to (128.8, 52.2)
Connections:
- net +5VA renamed +12VA
- U7 pad 3: (no net) -> unconnected-(U7-NC-Pad3)
Routing:
- net RIG_AF_OUT-: track 15.5 -> 30.9 mm
- net Net-(R25-Pad1): track 12.1 -> 18.2 mm
- net Net-(D2-COM): track 10.2 -> 13.3 mm
- net RIG_AF_OUT+: track 14.2 -> 16.3 mm
- net Net-(C11-Pad2): track 47.3 -> 49.4 mm
- net GNDA: track 23.4 -> 25.4 mm, vias 141 -> 143
- net Net-(Q1-G): track 12.1 -> 13.6 mm
Other:
- board text added: "KC1FSZ bruce@mackinnon.com"
- board text added: "MicroLink V4 2025-09"
- board text removed: "MicroLink V4 2025-09 KC1FSZ"
